File: hardware/kicad/Microphone.kicad_sch (KiCad schematic)
At the start: 24 parts, among them J1 POWER IN - 5V, J2 AUDIO OUT, U1 OPA1652D

Commit message: Update microphone preamplifier PCB layout and schematic
Parts:
- U1: symbol AudioPreamp:OPA1652D -> Amplifier_Operational:OPA1656ID
Changed lines of the file:
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@@
 		(rev "A")
 		(comment 1 "5 V single supply | Adjustable 30-40 dB gain")
-		(comment 2 "Designed by Ahmed Yehia Mohamed")
 	)
 	(text "AUDIO SIGNAL PATH"
@@
 	)
 	(symbol
-		(lib_id "AudioPreamp:OPA1652D")
+		(lib_id "Amplifier_Operational:OPA1656ID")
 		(at 111.76 38.1 0)
 		(unit 3)
@@
 	)
 	(symbol
-		(lib_id "AudioPreamp:OPA1652D")
+		(lib_id "Amplifier_Operational:OPA1656ID")
 		(at 190.5 40.64 0)
 		(mirror x)
@@
 	)
 	(symbol
-		(lib_id "AudioPreamp:OPA1652D")
+		(lib_id "Amplifier_Operational:OPA1656ID")
 		(at 166.37 100.33 0)
 		(mirror x)

Commit message: Sync KiCad sources to manufactured AD8656 revision
Parts:
- removed U1: OPA1652D, Package_SO:SOIC-8_3.9x4.9mm_P1.27mm, symbol Amplifier_Operational:OPA1656ID
- added D1: LED, LED_SMD:LED_1206_3216Metric, symbol Device:LED
- added R9: 2.2k, Resistor_SMD:R_0603_1608Metric_Pad0.98x0.95mm_HandSolder, symbol Device:R
- added SW1: SW_SPDT, AudioPreamp:SW_ESP1010_SPDT_Vertical, symbol Switch:SW_SPDT
- added U1: AD8656, Package_SO:MSOP-8_3x3mm_P0.65mm, symbol Amplifier_Operational:AD8656
Connections:
- net +5V: now also R9.1, SW1.1 (A), U1.8 (V+); no longer J1.1 (Pin_1)
- net AMP_OUT: now also U1.1
- net GND: now also MK1.2 (-), D1.1 (K), U1.4 (V-); no longer MK1.1 (-)
- net MIC_OUT: now also MK1.1 (+); no longer MK1.2 (+)
- net VBIAS: now also U1.3 (+)
- net VREF: now also U1.6 (-), U1.7
- net VREF_RAW: now also U1.5 (+)
- net at R5.1, R6.1: now also U1.2 (-)
- new net: J1.1 (Pin_1), SW1.2 (B)
- new net: D1.2 (A), R9.2
- no-connect marks 0 -> 1
Other:
- moved on the sheet: C1, C2, J1
